File: QL_CST_SCSI.kicad_pcb (KiCad board)
At the start: 2 copper layers, 125.7 x 97.8 mm, 44 parts, among them J1 QL_SLOT_DIN41612_CARD, J2 SCSI, J3 Floppy, Q1 PN2222A, U1 7805, U10 WD1770, U11 LS174, U12 74LS244, U13 74LS638, U14 74LS04, U15 74LS05, U16 GAL16V8, U2 LS266, U4 LS11, U5 LS245, U7 LS00, U8 LS240, U9 27C128, Y1 8Mhz

Commit message: small update
Connections:
- U15 pad 9: unconnected-(U15-Pad9) -> +5V
Routing:
- net (no net): track 0.00 -> 46.8 mm
- net +9V: track 15.3 -> 37.1 mm
- net unconnected-(U7-Pad13): track 0.00 -> 17.8 mm
- net unconnected-(U7-Pad12): track 0.00 -> 17.5 mm
- net unconnected-(U12-OEb-Pad19): track 0.00 -> 5.61 mm
- net unconnected-(U14-Pad9): track 0.00 -> 4.49 mm
- net GND: track 66.0 -> 68.7 mm
- net /RW: track 259.3 -> 258.2 mm
- net /A12: track 97.8 -> 96.9 mm
- net /SP2: track 39.7 -> 39.1 mm
