File: QL_CST_SCSI.kicad_sch (KiCad schematic)
At the start: 46 parts, among them J1 QL_SLOT_DIN41612_CARD, J2 SCSI, J3 Floppy, Q1 PN2222A, U1 7805, U10 WD1770, U11 LS174, U12 74LS244, U13 74LS638, U14 74LS04, U15 74LS05, U16 GAL16V8, U2 LS266, U3 LS03, U4 LS11, U5 LS245, U6 LS04, U7 LS00, U8 LS240, U9 27C128, Y1 8Mhz

Commit message: update
Parts:
- removed U3: LS03, Package_DIP:DIP-14_W7.62mm_Socket, symbol 74xx:74LS03
- removed U6: LS04, Package_DIP:DIP-14_W7.62mm_Socket, symbol 74xx:74LS04
- RP1: symbol Device:R_Pack04_SIP -> Device:R_Network07
Connections:
- net +5V: now also C9.2; no longer RP1.3 (R2.1)
- net A11: now also U4.3
- net A12: now also U4.2; no longer U4.3
- net A13: now also U4.1; no longer U4.2
- net A2: no longer U4.1
- net A3: no longer U7.5
- net D0: no longer U11.14 (D5)
- net D1: no longer U11.13 (D4)
- net D2: no longer U11.11 (D3)
- net D3: no longer U11.6 (D2)
- net D4: no longer U11.4 (D1)
- net D5: no longer U11.3 (D0)
- net DATA_RD: now also RP2.5 (R4); no longer RP2.4 (R3)
- net DATA_WR: no longer U8.14 (O2a)
- net DIR: no longer U8.16 (O1a)
- net DS0: no longer U8.12 (O3a)
- net DS1: no longer U8.9 (O0b)
- net FDC_WD: no longer U8.6 (I2a)
- net FDSET_CS: no longer U7.8
- net GATE_WR: no longer U8.5 (O2b)
- net GND: no longer U8.19 (OEb)
- net HEAD: no longer U8.3 (O3b)
- net MOTOR_ON: no longer U8.7 (O1b)
- net ROM_OE: no longer U14.11, U16.1 (I1/CLK), U7.13
- net SCSI_ACK: now also RP2.3 (R2)
- net SCSI_BUSY: now also RP2.2 (R1)
- net SCSI_SEL: now also RP2.4 (R3)
- net STEP: no longer U8.18 (O0a)
- net WRITE_PROT: now also RP2.8 (R7); no longer RP2.5 (R4)
- net XOR_PULLUP: now also RP1.2 (R1); no longer RP2.2 (R1)
- net interface_Sel: no longer RP1.2 (R1.2), RP1.4 (R2.2)
- net at U14.3: now also C17.1, R2.2
- net at U14.4: now also C8.1, R2.1, U14.5, Y1.2
- net at RP1.5 (R4): now also C18.2, U15.6; no longer C9.2
- net at R1.1: now also U14.1, Y1.1
- net at R1.2: now also C17.2, U14.2
- net at RP1.7 (R6): no longer Y1.1
- net EXT_INT: now reaches J1.b3 (~{EXTINT})
- net A3N_PULLUP: no longer names the net of U7.2
- net A3N_PULLUP: no longer RP2.3 (R2)
- removed net NOSE_6: U4.6, U7.1, U7.4
- new net: U7.1, U7.6
- new net: U14.11, U16.1 (I1/CLK)
- new net RP1_4: RP1.4 (R3)
- now unconnected: U7.10, U7.9
- no-connect marks 33 -> 30
Other:
- moved on the sheet: C1, C10, C11, C12, C13, C14, C15, C16, C17, C18, C2, C3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

Commit message: update 2
Connections:
- net +5V: now also D1.2 (A), U11.14 (D5)
- net GND: no longer J2.17 (Pin_17)
- net at D1.1 (K): now also J2.17 (Pin_17)
Other:
- moved on the sheet: C17, D1, R1, U14A, U14B, U15D, U15E, U7B, U7C, Y1

Commit message: small update
Connections:
- net +5V: now also U15.9
Other:
- title: CST Q-Disc Interface Version 4 -> CST SCSI-Disc Interface
- moved on the sheet: U15D
Changed lines of the file:
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@@
 	(paper "A2")
 	(title_block
-		(title "CST Q-Disc Interface Version 4")
-		(date "2023-05-20")
+		(title "CST SCSI-Disc Interface")
+		(date "2026-09-22")
 		(rev "00")
 		(company "Repro by Alvaro Alea Fdz.")
-		(comment 1 "To use with ROM Version 1.18")
-		(comment 2 "Disc Interface for Sinclair QL")
+		(comment 1 "Floppy and Hard Disk Interface for Sinclair QL")
 	)
 	(text "XT MODE: 2-3  (Plain Cable , drives DS0, DS1)\nAT MODE: 1-2, 3-4 (Cross Cable, both drives DS1)"
@@
 	)
 	(symbol
+		(lib_id "power:+5V")
+		(at 234.95 317.5 0)
+		(mirror y)
+		(unit 1)
+		(exclude_from_sim no)
+		(in_bom yes)
+		(on_board yes)
+		(dnp no)
+		(fields_autoplaced yes)
+		(property "Reference" "#PWR015"
+			(at 234.95 321.31 0)
+			(effects
+				(font
+					(size 1.27 1.27)
+				)
+				(hide yes)
+			)
+		)
+		(property "Value" "+5V"
+			(at 234.95 312.42 0)
+			(effects
+				(font
+					(size 1.27 1.27)
+				)
+			)
+		)
+		(property "Footprint" ""
+			(at 234.95 317.5 0)
+			(effects
+				(font
+					(size 1.27 1.27)
+				)
+				(hide yes)
+			)
+		)
+		(property "Datasheet" ""
+			(at 234.95 317.5 0)
+			(effects
+				(font
+					(size 1.27 1.27)
+				)
+				(hide yes)
+			)
+		)
+		(property "Description" ""
+			(at 234.95 317.5 0)
+			(effects
+				(font
+					(size 1.27 1.27)
+				)
+			)
+		)
+		(pin "1"
+		)
+		(instances
+			(project "QL_CST_SCSI"
+				(path "/aecd9f77-969e-41c8-a7ad-8348a70f1d7d"
+					(reference "#PWR015")
+					(unit 1)
+				)
+			)
+		)
+	)
+	(symbol
 		(lib_id "8bits:74LS638")
 		(at 368.3 210.82 180)
@@
 	(symbol
 		(lib_id "74xx:74LS05")
-		(at 381 306.07 0)
+		(at 242.57 317.5 0)
 		(unit 4)
 		(exclude_from_sim no)
@@
 		(dnp no)
 		(property "Reference" "U15"
-			(at 381 297.18 0)
+			(at 242.57 308.61 0)
 			(effects
 				(font
@@
 		)
 		(property "Value" "74LS05"
-			(at 381 299.72 0)
+			(at 242.57 311.15 0)
 			(effects
 				(font
@@
 		)
 		(property "Footprint" "Package_DIP:DIP-14_W7.62mm_Socket"
-			(at 381 306.07 0)
+			(at 242.57 317.5 0)
 			(effects
 				(font
@@
 		)
 		(property "Datasheet" "http://www.ti.com/lit/gpn/sn74LS05"
-			(at 381 306.07 0)
+			(at 242.57 317.5 0)
 			(effects
 				(font
@@
 		)
 		(property "Description" "Inverter Open Collect"
-			(at 381 306.07 0)
+			(at 242.57 317.5 0)
 			(effects
 				(font
